Commit message: "Core URDF Changes"

File: description/robot_core.xacro (robot description, xacro)
@@ -12,5 +12,5 @@
     </material>
     <material name="black">
-        <color rgba="0 0 0 1"/>
+        <color rgba="0 0 0 0.7"/>
     </material>
     <!-- BASE LINK -->
@@ -21,26 +21,80 @@
         <parent link="base_link"/>
         <child link="chassis"/>
-        <origin xyz="-0.21 0 0"/>
+        <origin xyz="-0.19 0 0"/>
     </joint>
     <link name="chassis">
         <visual>
-            <origin xyz="0.21 0 0"/>
-            <geometry>
-                <box size="0.5 0.5 0.02"/>
-            </geometry>
-            <material name="white"/>
-        </visual>
-        <collision>
-            <origin xyz="0.21 0 0"/>
-            <geometry>
-                <box size="0.5 0.5 0.02"/>
+            <origin xyz="0.19 0 0"/>
+            <geometry>
+                <box size="0.38 0.02 0.02"/>
+            </geometry>
+            <material name="black"/>
+        </visual>
+        <collision>
+            <origin xyz="0.19 0 0"/>
+            <geometry>
+                <box size="0.38 0.02 0.02"/>
             </geometry>
         </collision>
         <xacro:inertial_box mass="0.5" x="0.5" y="0.5" z="0.02">
-            <origin xyz="0.21 0 0.01" rpy="0 0 0"/>
+            <origin xyz="0.19 0 0.01" rpy="0 0 0"/>
         </xacro:inertial_box>
     </link>
     <gazebo reference="chassis">
-       <material>Gazebo/White</material>
+       <material>Gazebo/Black</material>
+    </gazebo>
+  <!-- FRONT CHASSIS LINK -->
+    <joint name="front_chassis_joint" type="fixed">
+        <parent link="base_link"/>
+        <child link="front_chassis"/>
+        <origin xyz="0.2 0 0"/>
+    </joint>
+    <link name="front_chassis">
+        <visual>
+            <origin xyz="0 0 0"/>
+            <geometry>
+                <box size="0.02 0.4 0.02"/>
+            </geometry>
+            <material name="black"/>
+        </visual>
+        <collision>
+            <origin xyz="0 0 0"/>
+            <geometry>
+                <box size="0.02 0.4 0.02"/>
+            </geometry>
+        </collision>
+        <xacro:inertial_box mass="0.5" x="0.5" y="0.5" z="0.02">
+            <origin xyz="0 0 0.01" rpy="0 0 0"/>
+        </xacro:inertial_box>
+    </link>
+    <gazebo reference="front_chassis">
+       <material>Gazebo/Black</material>
+    </gazebo>
+     <!--BACK CHASSIS LINK -->
+    <joint name="back_chassis_joint" type="fixed">
+        <parent link="base_link"/>
+        <child link="back_chassis"/>
+        <origin xyz="-0.2 0 0"/>
+    </joint>
+    <link name="back_chassis">
+        <visual>
+            <origin xyz="0 0 0"/>
+            <geometry>
+                <box size="0.02 0.4 0.02"/>
+            </geometry>
+            <material name="black"/>
+        </visual>
+        <collision>
+            <origin xyz="0 0 0"/>
+            <geometry>
+                <box size="0.02 0.4 0.02"/>
+            </geometry>
+        </collision>
+        <xacro:inertial_box mass="0.5" x="0.5" y="0.5" z="0.02">
+            <origin xyz="0 0 0.01" rpy="0 0 0"/>
+        </xacro:inertial_box>
+    </link>
+    <gazebo reference="back_chassis">
+       <material>Gazebo/Black</material>
     </gazebo>
      <!-- ROBOT BASE LINK -->
@@ -167,5 +221,5 @@
             <origin xyz="0 0 0"/>
             <geometry>
-                <box size="0.2 0.2 0.001"/>
+                <box size="0.1 0.1 0.001"/>
             </geometry>
             <material name="white"/>
@@ -174,5 +228,5 @@
             <origin xyz="0 0 0"/>
             <geometry>
-                <box size="0.2 0.2 0.001"/>
+                <box size="0.1 0.1 0.001"/>
             </geometry>
         </collision>
@@ -215,5 +269,5 @@
         <parent link="chassis"/>
         <child link="left_wheel"/>
-        <origin xyz="0 0.24 -0.06" rpy="-${pi/2} 0 0"/>
+        <origin xyz="0 0.19 -0.04" rpy="-${pi/2} 0 0"/>
         <axis xyz="0 0 1"/>
     </joint>
@@ -221,5 +275,5 @@
         <visual>
             <geometry>
-                <cylinder radius="0.04" length="0.02"/>
+                <cylinder radius="0.02" length="0.02"/>
             </geometry>
             <material name="blue"/>
@@ -227,8 +281,8 @@
         <collision>
             <geometry>
-                <cylinder radius="0.04" length="0.02"/>
-            </geometry>
-        </collision>
-        <xacro:inertial_cylinder mass="0.1" length="0.02" radius="0.04">
+                <cylinder radius="0.02" length="0.02"/>
+            </geometry>
+        </collision>
+        <xacro:inertial_cylinder mass="0.1" length="0.02" radius="0.02">
             <origin xyz="0 0 0" rpy="0 0 0"/>
         </xacro:inertial_cylinder>
@@ -241,5 +295,5 @@
         <parent link="chassis"/>
         <child link="right_wheel"/>
-        <origin xyz="0 -0.24 -0.06" rpy="${pi/2} 0 0" />
+        <origin xyz="0 -0.19 -0.04" rpy="${pi/2} 0 0" />
         <axis xyz="0 0 -1"/>
     </joint>
@@ -247,5 +301,5 @@
         <visual>
             <geometry>
-                <cylinder radius="0.04" length="0.02"/>
+                <cylinder radius="0.02" length="0.02"/>
             </geometry>
             <material name="blue"/>
@@ -253,8 +307,8 @@
         <collision>
             <geometry>
-                <cylinder radius="0.04" length="0.02"/>
-            </geometry>
-        </collision>
-        <xacro:inertial_cylinder mass="0.1" length="0.02" radius="0.04">
+                <cylinder radius="0.02" length="0.02"/>
+            </geometry>
+        </collision>
+        <xacro:inertial_cylinder mass="0.1" length="0.02" radius="0.02">
             <origin xyz="0 0 0" rpy="0 0 0"/>
         </xacro:inertial_cylinder>
@@ -267,10 +321,10 @@
         <parent link="base_link"/>
         <child link="caster_wheel1"/>
-        <origin xyz="0.21 -0.24 -0.06"/>
+        <origin xyz="0.20 -0.2 -0.04"/>
     </joint>
     <link name="caster_wheel1">
         <visual>
             <geometry>
-                <sphere radius="0.04"/>
+                <sphere radius="0.02"/>
             </geometry>
             <material name="blue"/>
@@ -278,8 +332,8 @@
         <collision>
             <geometry>
-                <sphere radius="0.04"/>
-            </geometry>
-        </collision>
-        <xacro:inertial_sphere mass="0.1" radius="0.04">
+                <sphere radius="0.02"/>
+            </geometry>
+        </collision>
+        <xacro:inertial_sphere mass="0.1" radius="0.02">
             <origin xyz="0 0 0" rpy="0 0 0"/>
         </xacro:inertial_sphere>
@@ -294,10 +348,10 @@
         <parent link="base_link"/>
         <child link="caster_wheel2"/>
-        <origin xyz="0.21 0.24 -0.06"/>
+        <origin xyz="0.2 0.2 -0.04"/>
     </joint>
     <link name="caster_wheel2">
         <visual>
             <geometry>
-                <sphere radius="0.04"/>
+                <sphere radius="0.02"/>
             </geometry>
             <material name="blue"/>
@@ -305,8 +359,8 @@
         <collision>
             <geometry>
-                <sphere radius="0.04"/>
-            </geometry>
-        </collision>
-        <xacro:inertial_sphere mass="0.1" radius="0.04">
+                <sphere radius="0.02"/>
+            </geometry>
+        </collision>
+        <xacro:inertial_sphere mass="0.1" radius="0.02">
             <origin xyz="0 0 0" rpy="0 0 0"/>
         </xacro:inertial_sphere>
